Commit message: add depth

File: gazebo/gazebo_plugins.xacro (robot description, xacro)
@@ -78,5 +78,5 @@
   </xacro:macro>
   <!-- -->
-  <xacro:macro name="add_gazebo_camera" params="link_name camera_name=camera frame:=camera_frame pose:='0 0 0 0 0 0' xyz:='0 0 0' rpy:='0 0 0' rate:=30.0 width:=800 height:=600 fov:=1.578" >
+  <xacro:macro name="add_gazebo_camera" params="link_name camera_name:=camera_n frame:=camera_frame pose:='0 0 0 0 0 0' xyz:='0 0 0' rpy:='0 0 0' rate:=30.0 width:=800 height:=600 fov:=1.578" >
     <!-- create camera frame-->
     <link name="${frame}" />
@@ -101,5 +101,5 @@
           </image>
           <clip>
-            <near>0.02</near>
+            <near>10</near>
             <far>300</far>
           </clip>
@@ -131,5 +131,5 @@
   </xacro:macro>
   <!-- -->
-  <xacro:macro name="add_gazebo_depth_camera" params="link_name camera_name frame:=depth_frame pose:='0 0 0 0 0 0' xyz:='0 0 0' rpy:='0 0 0' rate:=30.0 width:=800 height:=600 fov:=1.578" >
+  <xacro:macro name="add_gazebo_depth_camera" params="link_name camera_name:=depth_camera_n frame:=depth_frame pose:='0 0 0 0 0 0' xyz:='0 0 0' rpy:='0 0 0' rate:=30.0 width:=800 height:=600 fov:=1.578" >
     <!-- create camera frame-->
     <link name="${frame}" />
@@ -137,8 +137,9 @@
       <parent link="${link_name}"/>
       <child link="${frame}"/>
-      <origin xyz="${xyz}" rpy="${rpy}"/>
+      <origin xyz="-0.01 0 0" rpy="0 0 -1.578"/>
+      <!-- <origin xyz="${xyz}" rpy="${rpy}"/> -->
     </joint>
     <gazebo reference="${link_name}">
-      <sensor name="${link_nake}_depth_camera" type="depth">
+      <sensor name="${link_name}_depth_camera" type="depth">
         <pose>${pose}</pose>
         <always_on>true</always_on>
@@ -152,5 +153,5 @@
             <format>R8G8B8</format>
           </image>
-          <clip near="0.01" far="100.0" />
+          <clip near="1" far="100.0" />
           <save enabled="false" path="/tmp" />
           <depth_camera output="points" />

Commit message: add parts

File: gazebo/gazebo_plugins.xacro (robot description, xacro)
@@ -137,6 +137,5 @@
       <parent link="${link_name}"/>
       <child link="${frame}"/>
-      <origin xyz="-0.01 0 0" rpy="0 0 -1.578"/>
-      <!-- <origin xyz="${xyz}" rpy="${rpy}"/> -->
+      <origin xyz="${xyz}" rpy="${rpy}"/>
     </joint>
     <gazebo reference="${link_name}">

Commit message: 1.added camera_name to the macro 'add_depth_camera' 2.fixed spelling mistake

File: gazebo/gazebo_plugins.xacro (robot description, xacro)
@@ -138,5 +138,5 @@
   </xacro:macro>
   <!-- -->
-  <xacro:macro name="add_gazebo_depth_camera" params="link_name camera_name frame:=depth_frame pose:='0 0 0 0 0 0' xyz:='0 0 0' rpy:='0 0 0' rate:=30.0 width:=800 height:=600 fov:=1.578" >
+  <xacro:macro name="add_gazebo_depth_camera" params="link_name camera_name=depth_cam frame:=depth_frame pose:='0 0 0 0 0 0' xyz:='0 0 0' rpy:='0 0 0' rate:=30.0 width:=800 height:=600 fov:=1.578" >
     <!-- create camera frame-->
     <link name="${frame}" />
@@ -147,5 +147,5 @@
     </joint>
     <gazebo reference="${link_name}">
-      <sensor name="${link_nake}_depth_camera" type="depth">
+      <sensor name="${link_name}_depth_camera" type="depth">
         <pose>${pose}</pose>
         <always_on>true</always_on>

Commit message: b

File: gazebo/gazebo_plugins.xacro (robot description, xacro)
@@ -138,5 +138,5 @@
   </xacro:macro>
   <!-- -->
-  <xacro:macro name="add_gazebo_depth_camera" params="link_name camera_name:=depth_camera_n frame:=depth_frame pose:='0 0 0 0 0 0' xyz:='0 0 0' rpy:='0 0 0' rate:=30.0 width:=800 height:=600 fov:=1.578" >
+  <xacro:macro name="add_gazebo_depth_camera" params="link_name camera_name:=depth_camera frame:=depth_frame pose:='0 0 0 0 0 0' xyz:='0 0 0' rpy:='0 0 0' rate:=30.0 width:=800 height:=600 fov:=1.578" >
     <!-- create camera frame-->
     <link name="${frame}" />
@@ -144,5 +144,5 @@
       <parent link="${link_name}"/>
       <child link="${frame}"/>
-      <origin xyz="-0.01 0 0" rpy="0 0 -1.578"/>
+      <origin xyz="-0.01 0 0" rpy="-1.578 0 -1.578"/>
       <!-- <origin xyz="${xyz}" rpy="${rpy}"/> -->
     </joint>
@@ -160,5 +160,5 @@
             <format>R8G8B8</format>
           </image>
-          <clip near="1" far="100.0" />
+          <clip near="0.01" far="100.0" />
           <save enabled="false" path="/tmp" />
           <depth_camera output="points" />
